File: pcb/pcb_v1.2/BlinkStickAdvanced.kicad_sch (KiCad schematic)
At the start: 29 parts, among them J1 POWER, J2 USB_B_Micro, J3 ADD_HEADER_B, J4 ADD_HEADER_G, J5 ADD_HEADER_R, J6 RGB_HEADER, J7 RGB_HEADER, Q1 IRLR8726, Q2 IRLR8726, Q3 IRLR8726, U1 ATmega8-16A, Y1 Crystal_GND2_Small

Commit message: Move old PCB files to a different folder.
Parts:
- removed J1: POWER, TerminalBlock_Phoenix:TerminalBlock_Phoenix_MPT-0,5-4-2.54_1x04_P2.54mm_Horizontal, symbol Connector_Generic:Conn_01x04
- removed JP1: RST, symbol Jumper:Jumper_2_Open
- removed JP2: FLASH, symbol Jumper:SolderJumper_2_Open
- added C4: 1uF, Capacitor_SMD:C_0603_1608Metric_Pad1.08x0.95mm_HandSolder, symbol Device:C
- added J1: RST, Connector_PinHeader_2.54mm:PinHeader_1x02_P2.54mm_Vertical, symbol Connector_Generic:Conn_01x02
- added J3: FLASH, Connector_PinHeader_2.54mm:PinHeader_1x02_P2.54mm_Vertical, symbol Connector_Generic:Conn_01x02
- added J9: POWER, Connector_JST:JST_XH_B4B-XH-A_1x04_P2.50mm_Vertical, symbol Connector_Generic:Conn_01x04
- added TP1: GND, TestPoint:TestPoint_Pad_D1.5mm, symbol Connector:TestPoint
- added TP2: RXD, TestPoint:TestPoint_Pad_D1.5mm, symbol Connector:TestPoint
- added TP3: TXD, TestPoint:TestPoint_Pad_D1.5mm, symbol Connector:TestPoint
- renumbered C3 to C1, C1 to C2, C2 to C3, D2 to D1, D1 to D2, J3 to J4, J4 to J5, J5 to J6, J6 to J7, J7 to J8
Connections:
- net +12V: now also J9.4 (Pin_4)
- net +5V: now also C4.2
- net +5VA: now also J9.1 (Pin_1)
- net GND: now also C4.1, J1.1 (Pin_1), J3.1 (Pin_1), J9.2 (Pin_2), J9.3 (Pin_3), TP1.1
- net at U1.2 (PD4): now also J3.2 (Pin_2)
- net at U1.29 (PC6/~{RESET}): now also J1.2 (Pin_2)
- net RXD: now reaches U1.30 (PD0)
- net RXD: now also TP2.1
- net TXD: now reaches U1.31 (PD1)
- net TXD: now also TP3.1
- no-connect marks 18 -> 16
Other:
- moved on the sheet: J2
